Commit message: im a goddamned genious

File: inverse_kinematics/humanoid_3.urdf (robot description, URDF)
Before this commit: robot dumpUrdf, 40 links, 39 joints
Joints:
- joint chest_left_shoulder_joint1: axis 0 1 0 -> 0 0 1
- joint chest_left_shoulder_joint2: axis 0 0 1 -> 0 1 0
- joint chest_neck_joint1: axis 0 1 0 -> 0 0 1
- joint chest_neck_joint2: axis 0 0 1 -> 0 1 0
- joint chest_right_shoulder_joint1: axis 0 1 0 -> 0 0 1
- joint chest_right_shoulder_joint2: axis 0 0 1 -> 0 1 0
- joint left_knee_left_ankle_joint1: axis 0 1 0 -> 0 0 1
- joint left_knee_left_ankle_joint2: axis 0 0 1 -> 0 1 0
- joint right_knee_right_ankle_joint1: axis 0 1 0 -> 0 0 1
- joint right_knee_right_ankle_joint2: axis 0 0 1 -> 0 1 0
- joint root_chest_joint1: axis 0 1 0 -> 0 0 1
- joint root_chest_joint2: axis 0 0 1 -> 0 1 0
- joint root_left_hip_joint1: axis 0 1 0 -> 0 0 1
- joint root_left_hip_joint2: axis 0 0 1 -> 0 1 0
- joint root_right_hip_joint1: axis 0 1 0 -> 0 0 1
- joint root_right_hip_joint2: axis 0 0 1 -> 0 1 0
